File: logic/hardware_4850.kicad_pcb (KiCad board)
At the start: 4 copper layers, 84 x 79 mm, 202 parts, among them J101 PWM, J102 ADC, J1101 HALL, J1102 PWM_EN, J1103 CAN_IN, J1104 CAN_Out, J501 Enable, J601 AIN, J602 USB_B_Mini, J701 MOT_TEMP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

Commit message: .
Routing:
- net Net-(J1101-Pad4): track 25.0 -> 25.7 mm
