File: logic/interface.kicad_sch (KiCad schematic)
At the start: 27 parts

Commit message: start
Parts:
- gave numbers to parts that had none: 1
Changed lines of the file:
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@@
   (symbol (lib_id "Device:C") (at 99.06 87.63 0) (unit 1)
     (in_bom yes) (on_board yes)
-    (property "Reference" "" (id 0) (at 97.79 86.36 90)
+    (property "Reference" "U?" (id 0) (at 97.79 86.36 90)
       (effects (font (size 1.27 1.27)) (justify left))
     )
@@
   (symbol (lib_id "Device:C") (at 106.68 87.63 0) (unit 1)
     (in_bom yes) (on_board yes)
-    (property "Reference" "" (id 0) (at 105.41 86.36 90)
+    (property "Reference" "U?" (id 0) (at 105.41 86.36 90)
       (effects (font (size 1.27 1.27)) (justify left))
     )
@@
   (symbol (lib_id "Device:C") (at 121.92 87.63 0) (unit 1)
     (in_bom yes) (on_board yes)
-    (property "Reference" "" (id 0) (at 120.65 86.36 90)
+    (property "Reference" "U?" (id 0) (at 120.65 86.36 90)
       (effects (font (size 1.27 1.27)) (justify left))
     )
@@
   (symbol (lib_id "power:GNDD") (at 121.92 97.79 0) (unit 1)
     (in_bom yes) (on_board yes)
-    (property "Reference" "" (id 0) (at 121.92 104.14 0)
+    (property "Reference" "U?" (id 0) (at 121.92 104.14 0)
       (effects (font (size 1.27 1.27)) hide)
     )
@@
   (symbol (lib_id "Device:R") (at 64.77 66.04 270) (unit 1)
     (in_bom yes) (on_board yes)
-    (property "Reference" "" (id 0) (at 63.5 66.04 90)
+    (property "Reference" "U?" (id 0) (at 63.5 66.04 90)
       (effects (font (size 1.27 1.27)) (justify left))
     )
@@
   (symbol (lib_id "Device:R") (at 64.77 59.69 270) (unit 1)
     (in_bom yes) (on_board yes)
-    (property "Reference" "" (id 0) (at 63.5 59.69 90)
+    (property "Reference" "U?" (id 0) (at 63.5 59.69 90)
       (effects (font (size 1.27 1.27)) (justify left))
     )
@@
   (symbol (lib_id "Device:R") (at 64.77 53.34 270) (unit 1)
     (in_bom yes) (on_board yes)
-    (property "Reference" "" (id 0) (at 63.5 53.34 90)
+    (property "Reference" "U?" (id 0) (at 63.5 53.34 90)
       (effects (font (size 1.27 1.27)) (justify left))
     )
@@
   (symbol (lib_id "Device:R") (at 44.45 38.1 0) (unit 1)
     (in_bom yes) (on_board yes)
-    (property "Reference" "" (id 0) (at 44.45 39.37 90)
+    (property "Reference" "U?" (id 0) (at 44.45 39.37 90)
       (effects (font (size 1.27 1.27)) (justify left))
     )
@@
   (symbol (lib_id "Device:R") (at 49.53 38.1 0) (unit 1)
     (in_bom yes) (on_board yes)
-    (property "Reference" "" (id 0) (at 49.53 39.37 90)
+    (property "Reference" "U?" (id 0) (at 49.53 39.37 90)
       (effects (font (size 1.27 1.27)) (justify left))
     )
@@
   (symbol (lib_id "Device:R") (at 54.61 38.1 0) (unit 1)
     (in_bom yes) (on_board yes)
-    (property "Reference" "" (id 0) (at 54.61 39.37 90)
+    (property "Reference" "U?" (id 0) (at 54.61 39.37 90)
       (effects (font (size 1.27 1.27)) (justify left))
     )
@@
   (symbol (lib_id "Device:R") (at 39.37 38.1 0) (unit 1)
     (in_bom yes) (on_board yes)
-    (property "Reference" "" (id 0) (at 39.37 39.37 90)
+    (property "Reference" "U?" (id 0) (at 39.37 39.37 90)
       (effects (font (size 1.27 1.27)) (justify left))
     )
@@
   (symbol (lib_id "Device:C") (at 114.3 87.63 0) (unit 1)
     (in_bom yes) (on_board yes)
-    (property "Reference" "" (id 0) (at 113.03 86.36 90)
+    (property "Reference" "U?" (id 0) (at 113.03 86.36 90)
       (effects (font (size 1.27 1.27)) (justify left))
     )
@@
   (symbol (lib_id "Device:R") (at 64.77 46.99 270) (unit 1)
     (in_bom yes) (on_board yes)
-    (property "Reference" "" (id 0) (at 63.5 46.99 90)
+    (property "Reference" "U?" (id 0) (at 63.5 46.99 90)
       (effects (font (size 1.27 1.27)) (justify left))
     )
@@
   (symbol (lib_id "power:GNDA") (at 82.55 97.79 0) (unit 1)
     (in_bom yes) (on_board yes)
-    (property "Reference" "" (id 0) (at 82.55 104.14 0)
+    (property "Reference" "U?" (id 0) (at 82.55 104.14 0)
       (effects (font (size 1.27 1.27)) hide)
     )
@@
   (symbol (lib_id "Device:R") (at 82.55 38.1 0) (unit 1)
     (in_bom yes) (on_board yes)
-    (property "Reference" "" (id 0) (at 82.55 40.64 90)
+    (property "Reference" "U?" (id 0) (at 82.55 40.64 90)
       (effects (font (size 1.27 1.27)) (justify left))
     )
@@
   (symbol (lib_id "Device:C") (at 82.55 87.63 0) (mirror y) (unit 1)
     (in_bom yes) (on_board yes)
-    (property "Reference" "" (id 0) (at 83.82 86.36 90)
+    (property "Reference" "U?" (id 0) (at 83.82 86.36 90)
       (effects (font (size 1.27 1.27)) (justify left))
     )
@@
   (symbol (lib_id "Device:C") (at 124.46 171.45 0) (unit 1)
     (in_bom yes) (on_board yes)
-    (property "Reference" "" (id 0) (at 123.19 170.18 90)
+    (property "Reference" "U?" (id 0) (at 123.19 170.18 90)
       (effects (font (size 1.27 1.27)) (justify left))
     )
@@
   (symbol (lib_id "Device:R") (at 90.17 149.86 270) (unit 1)
     (in_bom yes) (on_board yes)
-    (property "Reference" "" (id 0) (at 88.9 149.86 90)
+    (property "Reference" "U?" (id 0) (at 88.9 149.86 90)
       (effects (font (size 1.27 1.27)) (justify left))
     )
@@
   (symbol (lib_id "power:GNDA") (at 107.95 181.61 0) (unit 1)
     (in_bom yes) (on_board yes)
-    (property "Reference" "" (id 0) (at 107.95 187.96 0)
+    (property "Reference" "U?" (id 0) (at 107.95 187.96 0)
       (effects (font (size 1.27 1.27)) hide)
     )
@@
   (symbol (lib_id "power:GNDD") (at 124.46 181.61 0) (unit 1)
     (in_bom yes) (on_board yes)
-    (property "Reference" "" (id 0) (at 124.46 187.96 0)
+    (property "Reference" "U?" (id 0) (at 124.46 187.96 0)
       (effects (font (size 1.27 1.27)) hide)
     )
@@
   (symbol (lib_id "Device:R") (at 64.77 140.97 0) (unit 1)
     (in_bom yes) (on_board yes)
-    (property "Reference" "" (id 0) (at 64.77 142.24 90)
+    (property "Reference" "U?" (id 0) (at 64.77 142.24 90)
       (effects (font (size 1.27 1.27)) (justify left))
     )
@@
   (symbol (lib_id "Device:R") (at 64.77 156.21 270) (unit 1)
     (in_bom yes) (on_board yes)
-    (property "Reference" "" (id 0) (at 63.5 156.21 90)
+    (property "Reference" "U?" (id 0) (at 63.5 156.21 90)
       (effects (font (size 1.27 1.27)) (justify left))
     )
@@
   (symbol (lib_id "Device:R") (at 64.77 162.56 270) (unit 1)
     (in_bom yes) (on_board yes)
-    (property "Reference" "" (id 0) (at 63.5 162.56 90)
+    (property "Reference" "U?" (id 0) (at 63.5 162.56 90)
       (effects (font (size 1.27 1.27)) (justify left))
     )
@@
   (symbol (lib_id "Device:R") (at 97.79 171.45 180) (unit 1)
     (in_bom yes) (on_board yes)
-    (property "Reference" "" (id 0) (at 97.79 170.18 90)
+    (property "Reference" "U?" (id 0) (at 97.79 170.18 90)
       (effects (font (size 1.27 1.27)) (justify left))
     )
@@
   (symbol (lib_id "Device:C") (at 107.95 171.45 0) (unit 1)
     (in_bom yes) (on_board yes)
-    (property "Reference" "" (id 0) (at 106.68 170.18 90)
+    (property "Reference" "U?" (id 0) (at 106.68 170.18 90)
       (effects (font (size 1.27 1.27)) (justify left))
     )
@@
   (symbol (lib_id "power:GNDD") (at 224.79 91.44 0) (mirror y) (unit 1)
     (in_bom yes) (on_board yes)
-    (property "Reference" "" (id 0) (at 224.79 97.79 0)
+    (property "Reference" "U?" (id 0) (at 224.79 97.79 0)
       (effects (font (size 1.27 1.27)) hide)
     )
@@
   (symbol (lib_id "power:+3V3") (at 224.79 41.91 0) (mirror y) (unit 1)
     (in_bom yes) (on_board yes)
-    (property "Reference" "" (id 0) (at 224.79 45.72 0)
+    (property "Reference" "U?" (id 0) (at 224.79 45.72 0)
       (effects (font (size 1.27 1.27)) hide)
     )
@@
   (symbol (lib_id "Device:C") (at 246.38 81.28 0) (mirror y) (unit 1)
     (in_bom yes) (on_board yes)
-    (property "Reference" "" (id 0) (at 247.65 80.01 90)
+    (property "Reference" "U?" (id 0) (at 247.65 80.01 90)
       (effects (font (size 1.27 1.27)) (justify left))
     )
@@
   (symbol (lib_id "Device:R") (at 208.28 143.51 90) (unit 1)
     (in_bom yes) (on_board yes)
-    (property "Reference" "" (id 0) (at 209.55 143.51 90)
+    (property "Reference" "U?" (id 0) (at 209.55 143.51 90)
       (effects (font (size 1.27 1.27)) (justify left))
     )
@@
   (symbol (lib_id "power:+3V3") (at 218.44 138.43 0) (mirror y) (unit 1)
     (in_bom yes) (on_board yes)
-    (property "Reference" "" (id 0) (at 218.44 142.24 0)
+    (property "Reference" "U?" (id 0) (at 218.44 142.24 0)
       (effects (font (size 1.27 1.27)) hide)
     )
@@
   (symbol (lib_id "Interface_CAN_LIN:SN65HVD230") (at 224.79 60.96 0) (mirror y) (unit 1)
     (in_bom yes) (on_board yes)
-    (property "Reference" "" (id 0) (at 227.33 49.53 0))
+    (property "Reference" "U?" (id 0) (at 227.33 49.53 0))
     (property "Value" "SN65HVD230" (id 1) (at 232.41 52.07 0))
     (property "Footprint" "Package_SO:SOIC-8_3.9x4.9mm_P1.27mm" (id 2) (at 224.79 73.66 0)
@@
       (effects (font (size 1.27 1.27)) hide)
     )
-    (property "LCSC#" "C12084" (id 4) (at 224.79 60.96 0)
-      (effects (font (size 1.27 1.27)) hide)
-    )
+    (property "LCSC#" "C12084" (id 4) (at 229.87 54.61 0))
     (pin "1")
     (pin "2")
@@
   (symbol (lib_id "Device:R") (at 259.08 66.04 270) (unit 1)
     (in_bom yes) (on_board yes)
-    (property "Reference" "" (id 0) (at 257.81 66.04 90)
+    (property "Reference" "U?" (id 0) (at 257.81 66.04 90)
       (effects (font (size 1.27 1.27)) (justify left))
     )
@@
   (symbol (lib_id "Device:R") (at 190.5 87.63 270) (unit 1)
     (in_bom yes) (on_board yes)
-    (property "Reference" "" (id 0) (at 190.5 87.63 90))
+    (property "Reference" "U?" (id 0) (at 190.5 87.63 90))
     (property "Value" "1R" (id 1) (at 195.58 86.36 90))
     (property "Footprint" "Resistor_SMD:R_0603_1608Metric" (id 2) (at 190.5 85.852 90)
