File: power/power_4850.kicad_pcb (KiCad board)
At the start: 4 copper layers, 104 x 79 mm, 302 parts, among them J1 +, J10 Enable, J11 CAN_IN, J12 CAN_OUT, J13 Debug, J2 Display, J3 A, J4 HALL, J5 B, J6 MOT_AUX, J7 C, J8 GND, J9 CRANK, P1 SWD, Q1 IPT015N10N5, Q2 IPT015N10N5, Q3 IPT015N10N5, Q4 IPT015N10N5, Q5 IPT015N10N5, Q6 IPT015N10N5, U1 1EDN7550B, U10 LM5008, U11 XC6206P332MR, U12 XC6206P332MR, U13 LMR12010X, U14 STM32G473VCTx, U15 SN65HVD230, U2 INA240A2PWR, U3 1EDN7550B, U4 1EDN7550B, U5 INA240A2PWR, U6 1EDN7550B, U7 1EDN7550B, U8 INA240A2PWR, U9 1EDN7550B, Y1 8MHz

Commit message: added supply connector for logic board
Parts:
- removed C1, C13, C16, C17, C2, C29, C32, C33, C45, C48, C49, C51, C57, C67, C68, C74, C75, C76, C79, C80, C81, C82, C83, C84, C85, C92, C93, C94, C95, C96: 100n, Capacitor_SMD:C_0603_1608Metric
- removed C10, C11, C12, C19, C20, C21, C22, C23, C24, C25, C26, C27, C28, C3, C35, C36, C37, C38, C39, C4, C40, C41, C42, C43, C44, C5, C56, C6, C7, C8, C9: 4u7, Capacitor_SMD:C_1210_3225Metric
- removed C14, C18, C30, C34, C46, C50, C54, C55, C60, C61, C62, C65, C77, C78: 10u, Capacitor_SMD:C_0805_2012Metric
- removed C15, C31, C47, C66, C72, C73: 10n, Capacitor_SMD:C_0603_1608Metric
- removed C52, C86, C87, C88, C89, C90, C91: 2n2, Capacitor_SMD:C_0603_1608Metric
- removed C53, C58, C59, C63, C64, C69: 1u, Capacitor_SMD:C_0603_1608Metric
- removed C70, C71: 15p, Capacitor_SMD:C_0603_1608Metric
- removed D1, D2, D3, D4, D5, D7, D8: SS210, Diode_SMD:D_SMA
- removed D10: RUN, LED_SMD:LED_0603_1608Metric
- removed D11: ERROR, LED_SMD:LED_0603_1608Metric
- removed D12: PWM, LED_SMD:LED_0603_1608Metric
- removed D13: ESDCAN24-2BLY, Package_TO_SOT_SMD:SOT-23
- removed D6: 12V, LED_SMD:LED_0603_1608Metric
- removed D9: 3V3, LED_SMD:LED_0603_1608Metric
- removed FB1, FB2, FB3, FB4, FB5, FB6, FB7, FB8, FB9: BLM18PG221SN1D, Resistor_SMD:R_0603_1608Metric
- removed H1, H2, H3: MountingHole_Pad, MountingHole:MountingHole_3.2mm_M3_Pad_Via
- removed J1: +, footprints:8X8X8.4MM TERMINAL
- removed J10: Enable, Connector_JST:JST_PH_B2B-PH-K_1x02_P2.00mm_Vertical
- removed J11: CAN_IN, Connector_JST:JST_PH_B4B-PH-K_1x04_P2.00mm_Vertical
- removed J12: CAN_OUT, Connector_JST:JST_PH_B4B-PH-K_1x04_P2.00mm_Vertical
- removed J13: Debug, Connector_USB:USB_Micro-B_Wuerth_614105150721_Vertical
- removed J2: Display, Connector_JST:JST_PH_B5B-PH-K_1x05_P2.00mm_Vertical
- removed J3: A, footprints:8X8X8.4MM TERMINAL
- removed J4: HALL, Connector_JST:JST_PH_B5B-PH-K_1x05_P2.00mm_Vertical
- removed J5: B, footprints:8X8X8.4MM TERMINAL
- removed J6: MOT_AUX, Connector_JST:JST_PH_B4B-PH-K_1x04_P2.00mm_Vertical
- removed J7: C, footprints:8X8X8.4MM TERMINAL
- removed J8: GND, footprints:8X8X8.4MM TERMINAL
- removed J9: CRANK, Connector_JST:JST_PH_B4B-PH-K_1x04_P2.00mm_Vertical
- removed JP1: BTLDR, Jumper:SolderJumper-2_P1.3mm_Open_RoundedPad1.0x1.5mm
- removed JP11: PBN-, NetTie:NetTie-2_SMD_Pad0.5mm
- removed JP13: PCN-, NetTie:NetTie-2_SMD_Pad0.5mm
- removed JP3: PA-, NetTie:NetTie-2_SMD_Pad0.5mm
- removed JP5: PB-, NetTie:NetTie-2_SMD_Pad0.5mm
- removed JP7: PC-, NetTie:NetTie-2_SMD_Pad0.5mm
- removed JP9: PAN-, NetTie:NetTie-2_SMD_Pad0.5mm
- removed L1: 330u, Inductor_SMD:L_Taiyo-Yuden_NR-80xx
- removed L2: 10u, Inductor_SMD:L_Taiyo-Yuden_NR-40xx
- removed N1: Housing, footprints:RND-455-00370
- removed P1: SWD, Connector_PinHeader_1.27mm:PinHeader_2x05_P1.27mm_Vertical
- removed Q1, Q2, Q3, Q4, Q5, Q6: IPT015N10N5, Package_TO_SOT_SMD:Infineon_PG-HSOF-8-1_ThermalVias
- removed R1, R11, R13, R15, R18, R20, R22, R24, R27, R29, R3, R4, R6, R69, R72, R9: 33k, Resistor_SMD:R_0603_1608Metric
- removed R10, R12, R14, R16, R19, R21, R23, R25, R28, R30, R5, R7, R701: 1R, Resistor_SMD:R_0603_1608Metric
- removed R17, R26, R8: R0002, footprints:R_5930_15076Metric_Pad5.20x8.75mm
- removed R2, R40, R42, R44, R45, R49, R50, R51, R52, R53, R54, R61, R62, R68, R71, R74: 1k, Resistor_SMD:R_0603_1608Metric
- removed R31: 220k, Resistor_SMD:R_0603_1608Metric
- removed R32: 2R2, Resistor_SMD:R_2512_6332Metric
- removed R33, R36, R43, R56, R57, R58, R59, R63, R64, R65, R66: 3k3, Resistor_SMD:R_0603_1608Metric
- removed R34, R39, R41, R55, R60, R67, R70, R73: 10k, Resistor_SMD:R_0603_1608Metric
- removed R35: 100k, Resistor_SMD:R_0603_1608Metric
- removed R37: 56k, Resistor_SMD:R_0603_1608Metric
- removed R38, R46, R47, R48: 470R, Resistor_SMD:R_0603_1608Metric
- removed TH1, TH2, TH3: NTC 10k, Resistor_SMD:R_0603_1608Metric
- removed TP1: IA_AC, TestPoint:TestPoint_Pad_D1.5mm
- removed TP2: IC_AC, TestPoint:TestPoint_Pad_D1.5mm
- removed TP3: IB_AC, TestPoint:TestPoint_Pad_D1.5mm
- removed U1, U3, U4, U6, U7, U9: 1EDN7550B, Package_TO_SOT_SMD:SOT-23-6
- removed U10: LM5008, Package_SO:MSOP-8_3x3mm_P0.65mm
- removed U11, U12: XC6206P332MR, Package_TO_SOT_SMD:SOT-23
- removed U13: LMR12010X, Package_TO_SOT_SMD:SOT-23-6
- removed U14: STM32G473VCTx, Package_QFP:LQFP-100_14x14mm_P0.5mm
- removed U15: SN65HVD230, Package_SO:SOIC-8_3.9x4.9mm_P1.27mm
- removed U2, U5, U8: INA240A2PWR, Package_SO:TSSOP-8_4.4x3mm_P0.65mm
- removed Y1: 8MHz, Crystal:Crystal_SMD_5032-2Pin_5.0x3.2mm
- added C219: 4u7, Capacitor_SMD:C_1210_3225Metric, F.Cu at (-68.6, 35.2)
- added C220: 4u7, Capacitor_SMD:C_1210_3225Metric, F.Cu at (-81.4, 41.6)
- added C221: DNP, Capacitor_SMD:C_0603_1608Metric, F.Cu at (-47.6, 41.6)
- added C222: DNP, Capacitor_SMD:C_0603_1608Metric, F.Cu at (-57.3, 50.1)
- added C223: 4u7, Capacitor_SMD:C_1210_3225Metric, F.Cu at (-68.6, 31.0)
- added C224: 4u7, Capacitor_SMD:C_1210_3225Metric, F.Cu at (-82.7, 54.4)
- added C225: 4u7, Capacitor_SMD:C_1210_3225Metric, F.Cu at (-75.8, 43.0)
- added C226: 4u7, Capacitor_SMD:C_1210_3225Metric, F.Cu at (-64.5, 43.8)
- added C227: 4u7, Capacitor_SMD:C_1210_3225Metric, F.Cu at (-70.1, 48.0)
- added C228: 4u7, Capacitor_SMD:C_1210_3225Metric, F.Cu at (-51.7, 30.7)
- added C229: 4u7, Capacitor_SMD:C_1210_3225Metric, F.Cu at (-57.3, 35.0)
- added C230: 4u7, Capacitor_SMD:C_1210_3225Metric, F.Cu at (-49.0, 26.4)
- added C231: 100n, Capacitor_SMD:C_0603_1608Metric, F.Cu at (-55.6, 42.6)
- added C232: 4u7, Capacitor_SMD:C_1210_3225Metric, F.Cu at (-77.0, 51.5)
- added C233: 4u7, Capacitor_SMD:C_1210_3225Metric, F.Cu at (-63.0, 39.2)
- added C234: 100n, Capacitor_SMD:C_0603_1608Metric, F.Cu at (-59.7, 45.1)
- added C235: 4u7, Capacitor_SMD:C_1210_3225Metric, F.Cu at (-70.1, 43.8)
- added C236: 4u7, Capacitor_SMD:C_1210_3225Metric, F.Cu at (-57.3, 30.7)
- added C237: 4u7, Capacitor_SMD:C_1210_3225Metric, F.Cu at (-63.0, 35.0)
- added C238: 4u7, Capacitor_SMD:C_1210_3225Metric, F.Cu at (-75.8, 47.2)
- added C319: 4u7, Capacitor_SMD:C_1210_3225Metric, F.Cu at (34.8, -17.7)
- added C320: 4u7, Capacitor_SMD:C_1210_3225Metric, F.Cu at (27.9, -9.63)
- added C321: DNP, Capacitor_SMD:C_0603_1608Metric, F.Cu at (67.8, -24.5)
- added C322: DNP, Capacitor_SMD:C_0603_1608Metric, F.Cu at (59.0, -16.0)
- added C323: 4u7, Capacitor_SMD:C_1210_3225Metric, F.Cu at (40.5, -16.4)
- added C324: 4u7, Capacitor_SMD:C_1210_3225Metric, F.Cu at (47.6, -32.6)
- added C325: 4u7, Capacitor_SMD:C_1210_3225Metric, F.Cu at (33.6, -9.23)
- added C326: 4u7, Capacitor_SMD:C_1210_3225Metric, F.Cu at (61.6, -37.2)
- added C327: 4u7, Capacitor_SMD:C_1210_3225Metric, F.Cu at (47.6, -24.1)
- added C328: 4u7, Capacitor_SMD:C_1210_3225Metric, F.Cu at (33.6, -13.5)
- added C329: 4u7, Capacitor_SMD:C_1210_3225Metric, F.Cu at (53.3, -32.9)
- added C330: 4u7, Capacitor_SMD:C_1210_3225Metric, F.Cu at (42.0, -29.1)
- added C331: 100n, Capacitor_SMD:C_0603_1608Metric, F.Cu at (68.6, -22.0)
- added C332: 4u7, Capacitor_SMD:C_1210_3225Metric, F.Cu at (47.6, -28.4)
- added C333: 4u7, Capacitor_SMD:C_1210_3225Metric, F.Cu at (55.9, -37.2)
- added C334: 100n, Capacitor_SMD:C_0603_1608Metric, F.Cu at (60.6, -18.5)
- added C335: 4u7, Capacitor_SMD:C_1210_3225Metric, F.Cu at (34.8, -22.0)
- added C336: 4u7, Capacitor_SMD:C_1210_3225Metric, F.Cu at (50.3, -37.2)
- added C337: 4u7, Capacitor_SMD:C_1210_3225Metric, F.Cu at (27.9, -13.9)
- added C338: 4u7, Capacitor_SMD:C_1210_3225Metric, F.Cu at (42.0, -24.9)
- added C419: 4u7, Capacitor_SMD:C_1210_3225Metric, F.Cu at (199.6, -45.8)
- added C420: 4u7, Capacitor_SMD:C_1210_3225Metric, F.Cu at (205.2, -50.0)
- added C421: DNP, Capacitor_SMD:C_0603_1608Metric, F.Cu at (210.3, -41.1)
- added C422: DNP, Capacitor_SMD:C_0603_1608Metric, F.Cu at (212.4, -43.6)
- added C423: 4u7, Capacitor_SMD:C_1210_3225Metric, F.Cu at (220.7, -67.3)
- added C424: 4u7, Capacitor_SMD:C_1210_3225Metric, F.Cu at (192.7, -42.2)
- added C425: 4u7, Capacitor_SMD:C_1210_3225Metric, F.Cu at (206.7, -54.5)
- added C426: 4u7, Capacitor_SMD:C_1210_3225Metric, F.Cu at (199.6, -50.0)
- added C427: 4u7, Capacitor_SMD:C_1210_3225Metric, F.Cu at (212.3, -63.0)
- added C428: 4u7, Capacitor_SMD:C_1210_3225Metric, F.Cu at (206.7, -58.8)
- added C429: 4u7, Capacitor_SMD:C_1210_3225Metric, F.Cu at (193.9, -46.5)
- added C430: 4u7, Capacitor_SMD:C_1210_3225Metric, F.Cu at (187.0, -39.4)
- added C431: 100n, Capacitor_SMD:C_0603_1608Metric, F.Cu at (208.4, -46.1)
- added C432: 4u7, Capacitor_SMD:C_1210_3225Metric, F.Cu at (201.1, -58.5)
- added C433: 4u7, Capacitor_SMD:C_1210_3225Metric, F.Cu at (215.0, -67.3)
- added C434: 100n, Capacitor_SMD:C_0603_1608Metric, F.Cu at (226.8, -63.5)
- added C435: 4u7, Capacitor_SMD:C_1210_3225Metric, F.Cu at (201.1, -54.2)
- added C436: 4u7, Capacitor_SMD:C_1210_3225Metric, F.Cu at (187.0, -43.6)
- added C437: 4u7, Capacitor_SMD:C_1210_3225Metric, F.Cu at (195.4, -59.2)
- added C438: 4u7, Capacitor_SMD:C_1210_3225Metric, F.Cu at (193.9, -50.8)
- added D201: 1N4148WS, Diode_SMD:D_SOD-323, F.Cu at (-52.4, 34.3)
- added D301: 1N4148WS, Diode_SMD:D_SOD-323, F.Cu at (63.9, -29.3)
- added D401: 1N4148WS, Diode_SMD:D_SOD-323, F.Cu at (217.3, -59.5)
- added H201: GND, MountingHole:MountingHole_3.2mm_M3_DIN965_Pad_TopOnly, F.Cu at (81.0, 62.5)
- added H202: Phase, MountingHole:MountingHole_3.2mm_M3, F.Cu at (118.0, 62.5)
- added H301: GND, MountingHole:MountingHole_3.2mm_M3_DIN965_Pad_TopOnly, F.Cu at (35.6, -27.7)
- added H302: Phase, MountingHole:MountingHole_3.2mm_M3, F.Cu at (21.1, -12.0)
- added H401: GND, MountingHole:MountingHole_3.2mm_M3_DIN965_Pad_TopOnly, F.Cu at (189.0, -57.8)
- added H402: Phase, MountingHole:MountingHole_3.2mm_M3, F.Cu at (174.6, -42.1)
- added J101: PA, Connector_PinSocket_2.54mm:PinSocket_2x05_P2.54mm_Vertical_SMD, F.Cu at (-29.5, 41.0)
- added J102: PB, Connector_PinSocket_2.54mm:PinSocket_2x05_P2.54mm_Vertical_SMD, F.Cu at (85.5, -27.0)
- added J103: PC, Connector_PinSocket_2.54mm:PinSocket_2x05_P2.54mm_Vertical_SMD, F.Cu at (239.5, -58.5)
- added J104: +, footprints:8X8X8.4MM TERMINAL, F.Cu at (240.0, -35.8)
- added J105: A, footprints:8X8X8.4MM TERMINAL, F.Cu at (94.2, 71.5)
- added J106: B, footprints:8X8X8.4MM TERMINAL, F.Cu at (72.8, -11.2)
- added J107: C, footprints:8X8X8.4MM TERMINAL, F.Cu at (184.3, -77.8)
- added J108: GND, footprints:8X8X8.4MM TERMINAL, F.Cu at (236.2, -15.8)
- added J109: Supply, Connector_PinSocket_2.54mm:PinSocket_2x02_P2.54mm_Vertical_SMD, F.Cu at (237.2, -26.0)
- added Q201: IPT015N10N5, Package_TO_SOT_SMD:Infineon_PG-HSOF-8-1_ThermalVias, F.Cu at (106.5, 61.8)
- added Q202: IPT015N10N5, Package_TO_SOT_SMD:Infineon_PG-HSOF-8-1_ThermalVias, F.Cu at (92.0, 61.8)
- added Q301: IPT015N10N5, Package_TO_SOT_SMD:Infineon_PG-HSOF-8-1_ThermalVias, F.Cu at (24.6, -21.8)
- added Q302: IPT015N10N5, Package_TO_SOT_SMD:Infineon_PG-HSOF-8-1_ThermalVias, F.Cu at (24.6, -33.5)
- added Q401: IPT015N10N5, Package_TO_SOT_SMD:Infineon_PG-HSOF-8-1_ThermalVias, F.Cu at (178.0, -52.0)
- added Q402: IPT015N10N5, Package_TO_SOT_SMD:Infineon_PG-HSOF-8-1_ThermalVias, F.Cu at (178.0, -63.6)
- added R201: 33k, Resistor_SMD:R_0603_1608Metric, F.Cu at (-57.3, 47.6)
- added R202: 33k, Resistor_SMD:R_0603_1608Metric, F.Cu at (-48.5, 39.1)
- added R203: 33k, Resistor_SMD:R_0603_1608Metric, F.Cu at (-51.6, 42.0)
- added R204: 33k, Resistor_SMD:R_0603_1608Metric, F.Cu at (-59.7, 42.6)
- added R205: 1R, Resistor_SMD:R_0603_1608Metric, F.Cu at (-52.5, 39.5)
- added R206: 1R, Resistor_SMD:R_0603_1608Metric, F.Cu at (-42.9, 30.2)
- added R207: 1R, Resistor_SMD:R_0603_1608Metric, F.Cu at (-48.3, 36.6)
- added R208: 1R, Resistor_SMD:R_0603_1608Metric, F.Cu at (-67.4, 54.7)
- added R209: 10R, Resistor_SMD:R_0603_1608Metric, F.Cu at (-61.3, 47.6)
- added R210: 10R, Resistor_SMD:R_0603_1608Metric, F.Cu at (-67.4, 52.1)
- added R211: 33k, Resistor_SMD:R_0603_1608Metric, F.Cu at (-48.3, 34.1)
- added R212: 1k, Resistor_SMD:R_0603_1608Metric, F.Cu at (-46.9, 30.2)
- added R213: 1k, Resistor_SMD:R_0603_1608Metric, F.Cu at (-52.5, 37.0)
- added R214: 1k, Resistor_SMD:R_0603_1608Metric, F.Cu at (-65.3, 49.6)
- added R215: 4k7, Resistor_SMD:R_0603_1608Metric, F.Cu at (-65.3, 47.1)
- added R216: 4k7, Resistor_SMD:R_0603_1608Metric, F.Cu at (-55.6, 45.1)
- added R217: 10k, Resistor_SMD:R_0603_1608Metric, F.Cu at (-61.3, 50.1)
- added R218: 10k, Resistor_SMD:R_0603_1608Metric, F.Cu at (-44.2, 32.7)
- added R301: 33k, Resistor_SMD:R_0603_1608Metric, F.Cu at (72.0, -28.4)
- added R302: 33k, Resistor_SMD:R_0603_1608Metric, F.Cu at (52.9, -8.50)
- added R303: 33k, Resistor_SMD:R_0603_1608Metric, F.Cu at (64.6, -19.1)
- added R304: 33k, Resistor_SMD:R_0603_1608Metric, F.Cu at (56.9, -11.0)
- added R305: 1R, Resistor_SMD:R_0603_1608Metric, F.Cu at (59.0, -13.5)
- added R306: 1R, Resistor_SMD:R_0603_1608Metric, F.Cu at (69.4, -33.4)
- added R307: 1R, Resistor_SMD:R_0603_1608Metric, F.Cu at (52.9, -11.0)
- added R308: 1R, Resistor_SMD:R_0603_1608Metric, F.Cu at (55.0, -16.0)
- added R309: 10R, Resistor_SMD:R_0603_1608Metric, F.Cu at (64.6, -21.6)
- added R310: 10R, Resistor_SMD:R_0603_1608Metric, F.Cu at (50.9, -16.5)
- added R311: 33k, Resistor_SMD:R_0603_1608Metric, F.Cu at (63.7, -24.1)
- added R312: 1k, Resistor_SMD:R_0603_1608Metric, F.Cu at (73.4, -33.4)
- added R313: 1k, Resistor_SMD:R_0603_1608Metric, F.Cu at (48.9, -8.97)
- added R314: 1k, Resistor_SMD:R_0603_1608Metric, F.Cu at (48.9, -11.5)
- added R315: 4k7, Resistor_SMD:R_0603_1608Metric, F.Cu at (68.0, -29.6)
- added R316: 4k7, Resistor_SMD:R_0603_1608Metric, F.Cu at (56.6, -21.1)
- added R317: 10k, Resistor_SMD:R_0603_1608Metric, F.Cu at (50.9, -14.0)
- added R318: 10k, Resistor_SMD:R_0603_1608Metric, F.Cu at (68.0, -27.0)
- added R401: 33k, Resistor_SMD:R_0603_1608Metric, F.Cu at (214.0, -48.7)
- added R402: 33k, Resistor_SMD:R_0603_1608Metric, F.Cu at (217.2, -54.2)
- added R403: 33k, Resistor_SMD:R_0603_1608Metric, F.Cu at (221.4, -57.2)
- added R404: 33k, Resistor_SMD:R_0603_1608Metric, F.Cu at (202.3, -39.1)
- added R405: 1R, Resistor_SMD:R_0603_1608Metric, F.Cu at (202.3, -41.6)
- added R406: 1R, Resistor_SMD:R_0603_1608Metric, F.Cu at (214.0, -51.2)
- added R407: 1R, Resistor_SMD:R_0603_1608Metric, F.Cu at (221.4, -59.7)
- added R408: 1R, Resistor_SMD:R_0603_1608Metric, F.Cu at (222.8, -63.5)
- added R409: 10R, Resistor_SMD:R_0603_1608Metric, F.Cu at (204.4, -44.1)
- added R410: 10R, Resistor_SMD:R_0603_1608Metric, F.Cu at (204.4, -46.6)
- added R411: 33k, Resistor_SMD:R_0603_1608Metric, F.Cu at (217.2, -56.7)
- added R412: 1k, Resistor_SMD:R_0603_1608Metric, F.Cu at (210.0, -51.2)
- added R413: 1k, Resistor_SMD:R_0603_1608Metric, F.Cu at (208.4, -43.6)
- added R414: 1k, Resistor_SMD:R_0603_1608Metric, F.Cu at (225.4, -61.0)
- added R415: 4k7, Resistor_SMD:R_0603_1608Metric, F.Cu at (218.1, -51.7)
- added R416: 4k7, Resistor_SMD:R_0603_1608Metric, F.Cu at (221.2, -54.6)
- added R417: 10k, Resistor_SMD:R_0603_1608Metric, F.Cu at (212.4, -46.1)
- added R418: 10k, Resistor_SMD:R_0603_1608Metric, F.Cu at (206.3, -41.1)
- added TH201: NTC 10k, Resistor_SMD:R_0603_1608Metric, F.Cu at (-51.6, 44.6)
- added TH301: NTC 10k, Resistor_SMD:R_0603_1608Metric, F.Cu at (63.7, -26.6)
- added TH401: NTC 10k, Resistor_SMD:R_0603_1608Metric, F.Cu at (218.1, -49.2)
- added U201: 1EDN7550B, Package_TO_SOT_SMD:SOT-23-6, F.Cu at (-43.8, 26.6)
- added U202: 1EDN7550B, Package_TO_SOT_SMD:SOT-23-6, F.Cu at (-71.8, 52.5)
- added U203: ACS72981KLATR-150B5, Sensor_Current:Allegro_PSOF-7_4.8x6.4mm_P1.60mm, F.Cu at (107.0, 71.0)
- added U204: MCP6D11-EMS, Package_SO:MSOP-8_3x3mm_P0.65mm, F.Cu at (121.0, 72.0)
- added U301: 1EDN7550B, Package_TO_SOT_SMD:SOT-23-6, F.Cu at (72.5, -37.0)
- added U302: 1EDN7550B, Package_TO_SOT_SMD:SOT-23-6, F.Cu at (44.5, -11.2)
- added U303: ACS72981KLATR-150B5, Sensor_Current:Allegro_PSOF-7_4.8x6.4mm_P1.60mm, F.Cu at (36.0, -35.3)
- added U304: MCP6D11-EMS, Package_SO:MSOP-8_3x3mm_P0.65mm, F.Cu at (43.7, -37.0)
- added U401: 1EDN7550B, Package_TO_SOT_SMD:SOT-23-6, F.Cu at (225.9, -67.1)
- added U402: 1EDN7550B, Package_TO_SOT_SMD:SOT-23-6, F.Cu at (197.9, -41.3)
- added U403: ACS72981KLATR-150B5, Sensor_Current:Allegro_PSOF-7_4.8x6.4mm_P1.60mm, F.Cu at (189.4, -65.4)
- added U404: MCP6D11-EMS, Package_SO:MSOP-8_3x3mm_P0.65mm, F.Cu at (197.2, -67.2)
- C201, C202, C213, C216, C301, C302, C313, C316, C401, C402, C413, C416: value 4u7 -> 100n; footprint Capacitor_SMD:C_1210_3225Metric -> Capacitor_SMD:C_0603_1608Metric
- C203, C204, C303, C304, C403, C404: value 4u7 -> 10u; footprint Capacitor_SMD:C_1210_3225Metric -> Capacitor_SMD:C_0805_2012Metric
- moved C218 198.2 mm to (-60.3, 26.4), turned to 0 degrees
- moved C211 196.0 mm to (-88.3, 49.8), turned to 0 degrees
- moved C217 186.8 mm to (-81.4, 45.9), turned to 0 degrees
- moved C413 183.5 mm to (222.1, -52.1), turned to 0 degrees
- moved C414 181.3 mm to (203.7, -67.3), turned to 0 degrees
- moved C412 180.6 mm to (206.7, -63.0), turned to 0 degrees
- moved C215 175.6 mm to (-88.3, 54.0), turned to 0 degrees
- moved C205 173.1 mm to (-74.3, 34.5), turned to 0 degrees
- moved C409 170.8 mm to (195.4, -55.0), turned to 0 degrees
- moved C203 167.7 mm to (-74.0, 30.4), turned to 0 degrees
- moved C206 166.9 mm to (-63.0, 30.7), turned to 0 degrees
- moved C405 166.3 mm to (209.4, -67.3), turned to 0 degrees
- moved C207 165.9 mm to (-82.7, 50.1), turned to 0 degrees
- moved C214 162.0 mm to (-57.3, 39.2), turned to 0 degrees
- moved C415 161.8 mm to (188.2, -52.1), turned to 0 degrees
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Connections:
- C201 pad 1: +BATT -> Net-(C201-Pad1)
- C201 pad 2: GNDPWR -> /phase_a/Phase+
- C202 pad 1: +BATT -> Net-(C202-Pad1)
- C203 pad 1: +BATT -> Net-(C201-Pad1)
- C203 pad 2: GNDPWR -> /phase_a/Phase+
- C204 pad 1: +BATT -> Net-(C202-Pad1)
- C213 pad 1: +BATT -> /phase_a/+5V
- C213 pad 2: GNDPWR -> /phase_a/GNDA
- C216 pad 1: +BATT -> Net-(C216-Pad1)
- C216 pad 2: GNDPWR -> /phase_a/GNDA
- C301 pad 1: +BATT -> Net-(C301-Pad1)
- C301 pad 2: GNDPWR -> /phase_b/Phase+
- C302 pad 1: +BATT -> Net-(C302-Pad1)
- C303 pad 1: +BATT -> Net-(C301-Pad1)
- C303 pad 2: GNDPWR -> /phase_b/Phase+
- C304 pad 1: +BATT -> Net-(C302-Pad1)
- C313 pad 1: +BATT -> /phase_b/+5V
- C313 pad 2: GNDPWR -> /phase_b/GNDA
- C316 pad 1: +BATT -> Net-(C316-Pad1)
- C316 pad 2: GNDPWR -> /phase_b/GNDA
- C401 pad 1: +BATT -> Net-(C401-Pad1)
- C401 pad 2: GNDPWR -> /phase_c/Phase+
- C402 pad 1: +BATT -> Net-(C402-Pad1)
- C403 pad 1: +BATT -> Net-(C401-Pad1)
- C403 pad 2: GNDPWR -> /phase_c/Phase+
- C404 pad 1: +BATT -> Net-(C402-Pad1)
- C413 pad 1: +BATT -> /phase_c/+5V
- C413 pad 2: GNDPWR -> /phase_c/GNDA
- C416 pad 1: +BATT -> Net-(C416-Pad1)
- C416 pad 2: GNDPWR -> /phase_c/GNDA
Routing:
- net GNDA: track 69.2 -> 0.00 mm, vias 26 -> 0
- net GNDD: track 45.2 -> 0.00 mm, vias 33 -> 0
- net +BATT: track 43.9 -> 0.00 mm, vias 373 -> 0
- net GNDPWR: track 39.0 -> 0.00 mm, vias 502 -> 0
- net Net-(C52-Pad1): track 36.6 -> 0.00 mm, vias 2 -> 0
- net /mcu/IC_AC_IN: track 32.5 -> 0.00 mm, vias 2 -> 0
- net +3V3: track 29.3 -> 0.00 mm, vias 10 -> 0
- net /mcu/IA_DC: track 24.0 -> 0.00 mm
- net /mcu/IB_DC: track 22.6 -> 0.00 mm
- net /Interface/VREF: track 20.7 -> 0.00 mm, vias 11 -> 0
- net /phase_c/Phase-: track 18.7 -> 0.00 mm
- net +3.3VADC: track 17.7 -> 0.00 mm, vias 1 -> 0
- net /mcu/AIN_IA: track 15.1 -> 0.00 mm, vias 2 -> 0
- net /mcu/IA_AC_IN: track 13.2 -> 0.00 mm
- net /power_supply/DCDC_VIN: track 12.7 -> 0.00 mm
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- removed copper zone on F.Cu, net +12V
- removed copper zone on B.Cu, net +3.3VADC
- removed copper zone on VCC, net +3V3
- removed copper zone on F.Cu, net +5V
- removed copper zone on B.Cu, net +BATT
- removed copper zone on F.Cu, net +BATT
- removed copper zone on VCC, net +BATT
- removed copper zone on VCC, net /Interface/VREF
- removed copper zone on F.Cu, net /phase_a/Phase+
- removed copper zone on F.Cu, net /phase_a/Phase-
- removed copper zone on F.Cu, net /phase_b/Phase+
- removed copper zone on F.Cu, net /phase_b/Phase-
- removed copper zone on F.Cu, net /phase_c/Phase+
- removed copper zone on F.Cu, net /phase_c/Phase-
- removed copper zone on F.Cu, net /power_supply/DCDC_VIN
- removed copper zone on GND, net GNDA
- removed copper zone on GND, net GNDD
- removed copper zone on F.Cu, net GNDPWR
- removed copper zone on GND, net GNDPWR
- removed copper zone on F.Cu, net Net-(C51-Pad1)
- removed copper zone on F.Cu, net Net-(C52-Pad1)
Other:
- board outline removed
